Commit message: Added the realsense camera to the gazebo package

File: rover_description/urdf/rover.xacro (robot description, xacro)
@@ -54,4 +54,5 @@
     <child link="left_rear_wheel" />
     <axis xyz="0 0 -1" />
+    <!--dynamics damping="0.05" friction="0.0"/-->
     <limit effort="10" velocity="100" />
   </joint>
@@ -75,4 +76,5 @@
     <child link="right_rear_wheel" />
     <axis xyz="0 0 -1" />
+    <!--dynamics damping="0.05" friction="0.0"/-->
     <limit effort="10" velocity="100" />
   </joint>
@@ -132,4 +134,5 @@
     <child link="left_front_wheel" />
     <axis xyz="0 0 -1" />
+    <!--dynamics damping="0.05" friction="0.0"/-->
     <limit effort="10" velocity="100" />
   </joint>
@@ -152,8 +155,48 @@
     <parent link="right_steering_hinge" />
     <child link="right_front_wheel" />
+    <!--dynamics damping="0.05" friction="0.0"/-->
     <axis xyz="0 0 -1" />
     <limit effort="10" velocity="100"/>
   </joint>
   <xacro:wheel_transmission name="right_front_wheel" />
+  <xacro:arg name="name" default="camera" />
+  <xacro:arg name="topics_ns" default="camera" />
+  <xacro:arg name="use_nominal_extrinsics" default="false" />
+  <xacro:arg name="publish_pointcloud" default="false" />
+  <xacro:arg name="add_plug" default="false" />
+  <xacro:include filename="$(find realsense2_description)/urdf/_d435.urdf.xacro" />
+  <link name="realsense"/>
+  <xacro:sensor_d435 name="$(arg name)" topics_ns="$(arg topics_ns)" parent="realsense" use_nominal_extrinsics="$(arg use_nominal_extrinsics)" publish_pointcloud="$(arg publish_pointcloud)" add_plug="$(arg add_plug)">
+    <origin xyz="0 0 0" rpy="0 0 0"/>
+  </xacro:sensor_d435>
+ <!--link name="realsense">
+   <inertial>
+     <mass value="1e-5" />
+     <origin xyz="0 0 0" rpy="0 0 0"/>
+     <inertia ixx="1e-6" ixy="0" ixz="0" iyy="1e-6" iyz="0" izz="1e-6" />
+   </inertial>
+   <collision>
+     <origin xyz="0 0 0" rpy="0 0 0"/>
+     <geometry>
+       <box size="0.033 0.175 0.030"/>
+     </geometry>
+   </collision>
+   <visual>
+     <origin xyz="0 0 0" rpy="0 0 0"/>
+     <geometry>
+       <mesh filename="package://realsense2_description/meshes/d435.dae"/>
+     </geometry>
+   </visual>
+ </link-->
+ <!--xacro:include filename="$(find realsense2_description)/urdf/_d435.urdf.xacro">
+   <sensor_d435 parent="realsense_link">
+   </sensor_d435>
+ </xacro:include-->
+ <joint name="realsense_joint" type="fixed">
+   <origin xyz="0.2 0.0 0.15" rpy="0 0 0"/>
+   <parent link="chassis" />
+   <child link="realsense" />
+   <axis xyz="0 0 1" />
+ </joint>
   <!-- Add Hokuyo laser scanner -->
   <link name="laser">
@@ -181,60 +224,4 @@
     <axis xyz="0 0 1" />
   </joint>
-  <!-- zed camera -->
-  <link name="zed_camera_link">
-    <inertial>
-      <mass value="1e-5" />
-      <origin xyz="0 0 0" rpy="0 0 0"/>
-      <inertia ixx="1e-6" ixy="0" ixz="0" iyy="1e-6" iyz="0" izz="1e-6" />
-    </inertial>
-    <collision>
-      <origin xyz="0 0 0" rpy="0 0 0"/>
-      <geometry>
-        <box size="0.033 0.175 0.030"/>
-      </geometry>
-    </collision>
-    <visual>
-      <origin xyz="0 0 0" rpy="0 0 0"/>
-      <geometry>
-        <box size="0.033 0.175 0.030"/>
-      </geometry>
-      <material name="red"/>
-    </visual>
-  </link>
-  <joint name="zed_camera_joint" type="fixed">
-    <origin xyz="0.25 0 0.04" rpy="0 0 0"/>
-    <parent link="chassis"/>
-    <child link="zed_camera_link"/>
-    <axis xyz="0 0 1" />
-    <!-- <limit lower="0.0" upper="0.0" effort="0.0" velocity="0.0" /> -->
-  </joint>
-  <!-- zed camera lenses -->
-  <!-- It seems these have to have a non-zero mass to have a camera attached? -->
-  <link name="camera_link"><!-- this needs to match the name in zed_wrapper/zed_tf.launch -->
-    <inertial>
-      <mass value="1e-5" />
-      <origin xyz="0 0 0" rpy="0 0 0"/>
-      <inertia ixx="1e-6" ixy="0" ixz="0" iyy="1e-6" iyz="0" izz="1e-6" />
-    </inertial>
-  </link>
-  <link name="zed_camera_right_link">
-    <inertial>
-      <mass value="1e-5" />
-      <origin xyz="0 0 0" rpy="0 0 0"/>
-      <inertia ixx="1e-6" ixy="0" ixz="0" iyy="1e-6" iyz="0" izz="1e-6" />
-    </inertial>
-  </link>
-  <joint name="zed_camera_left_joint" type="fixed">
-    <origin xyz="0 0.06 0" rpy="0 0 0"/>
-    <parent link="zed_camera_link"/>
-    <child link="camera_link"/>
-    <axis xyz="0 0 1" />
-  </joint>
-  <joint name="zed_camera_right_joint" type="fixed">
-    <origin xyz="0 -0.06 0" rpy="0 0 0"/>
-    <parent link="zed_camera_link"/>
-    <child link="zed_camera_right_link"/>
-    <axis xyz="0 0 1" />
-  </joint>
   <!-- Add the remaining xacros -->
   <xacro:include filename="$(find rover_description)/urdf/rover.gazebo" />

Commit message: Updated Rover Dynamics

File: rover_description/urdf/rover.xacro (robot description, xacro)
@@ -134,5 +134,5 @@
     <child link="left_front_wheel" />
     <axis xyz="0 0 -1" />
-    <!--dynamics damping="0.05" friction="0.0"/-->
+    <dynamics damping="0.005" friction="0.0"/>
     <limit effort="10" velocity="100" />
   </joint>
@@ -155,5 +155,5 @@
     <parent link="right_steering_hinge" />
     <child link="right_front_wheel" />
-    <!--dynamics damping="0.05" friction="0.0"/-->
+    <dynamics damping="0.005" friction="0.0"/>
     <axis xyz="0 0 -1" />
     <limit effort="10" velocity="100"/>

Commit message: added IMU functionality

File: rover_description/urdf/rover.xacro (robot description, xacro)
@@ -170,23 +170,4 @@
     <origin xyz="0 0 0" rpy="0 0 0"/>
   </xacro:sensor_d435>
- <!--link name="realsense">
-   <inertial>
-     <mass value="1e-5" />
-     <origin xyz="0 0 0" rpy="0 0 0"/>
-     <inertia ixx="1e-6" ixy="0" ixz="0" iyy="1e-6" iyz="0" izz="1e-6" />
-   </inertial>
-   <collision>
-     <origin xyz="0 0 0" rpy="0 0 0"/>
-     <geometry>
-       <box size="0.033 0.175 0.030"/>
-     </geometry>
-   </collision>
-   <visual>
-     <origin xyz="0 0 0" rpy="0 0 0"/>
-     <geometry>
-       <mesh filename="package://realsense2_description/meshes/d435.dae"/>
-     </geometry>
-   </visual>
- </link-->
  <!--xacro:include filename="$(find realsense2_description)/urdf/_d435.urdf.xacro">
    <sensor_d435 parent="realsense_link">
@@ -224,5 +205,30 @@
     <axis xyz="0 0 1" />
   </joint>
-  <!-- Add the remaining xacros -->
+<joint name="imu_joint" type="fixed">
+  <axis xyz="1 0 0"/> <!-- 0 1 0 -->
+  <origin xyz="0 0 0.19"/>
+  <parent link="base_link"/>
+  <child link="imu_link"/>
+</joint>
+<link name="imu_link">
+  <inertial>
+    <mass value="0.001"/>
+    <origin rpy="0 0 0" xyz="0 0 0"/>
+    <inertia ixx="0.0001" ixy="0" ixz="0" iyy="0.000001" iyz="0" izz="0.0001"/>
+  </inertial>
+  <visual>
+    <origin rpy="0 0 0" xyz="0 0 0"/>
+    <geometry>
+      <box size="0.001 0.001 0.001"/>
+    </geometry>
+  </visual>
+  <collision>
+    <origin rpy="0 0 0" xyz="0 0 0"/>
+    <geometry>
+      <box size=".001 .001 .001"/>
+    </geometry>
+  </collision>
+</link>
+  <!-- Ahttps://github.com/NevzatBOL/ROS-Beginner/blob/master/catkin_ws/src/sensor_models/urdf/imu.xmldd the remaining xacros -->
   <xacro:include filename="$(find rover_description)/urdf/rover.gazebo" />
   <xacro:include filename="$(find rover_description)/urdf/materials.xacro" />

Commit message: added GPS joint and link

File: rover_description/urdf/rover.xacro (robot description, xacro)
@@ -230,4 +230,29 @@
   </collision>
 </link>
+<joint name="gps_joint" type="fixed">
+  <axis xyz="1 0 0"/> <!-- 0 1 0 -->
+  <origin xyz="0 0 0.05"/>
+  <parent link="base_link"/>
+  <child link="gps_link"/>
+</joint>
+<link name="gps_link">
+  <inertial>
+    <mass value="0.001"/>
+    <origin rpy="0 0 0" xyz="0 0 0"/>
+    <inertia ixx="0.0001" ixy="0" ixz="0" iyy="0.000001" iyz="0" izz="0.0001"/>
+  </inertial>
+  <visual>
+    <origin rpy="0 0 0" xyz="0 0 0"/>
+    <geometry>
+      <box size="0.001 0.001 0.001"/>
+    </geometry>
+  </visual>
+  <collision>
+    <origin rpy="0 0 0" xyz="0 0 0"/>
+    <geometry>
+      <box size=".001 .001 .001"/>
+    </geometry>
+  </collision>
+</link>
   <!-- Ahttps://github.com/NevzatBOL/ROS-Beginner/blob/master/catkin_ws/src/sensor_models/urdf/imu.xmldd the remaining xacros -->
   <xacro:include filename="$(find rover_description)/urdf/rover.gazebo" />

Commit message: snapshot of last spring

File: rover_description/urdf/rover.xacro (robot description, xacro)
@@ -206,5 +206,4 @@
   </joint>
 <joint name="imu_joint" type="fixed">
-  <axis xyz="1 0 0"/> <!-- 0 1 0 -->
   <origin xyz="0 0 0.19"/>
   <parent link="base_link"/>
@@ -231,7 +230,6 @@
 </link>
 <joint name="gps_joint" type="fixed">
-  <axis xyz="1 0 0"/> <!-- 0 1 0 -->
   <origin xyz="0 0 0.05"/>
-  <parent link="base_link"/>
+  <parent link="imu_link"/>
   <child link="gps_link"/>
 </joint>

Commit message: Save old version of rover description

File: rover_description/urdf/rover.xacro (robot description, xacro)
@@ -4,8 +4,26 @@
   <!-- Add chassis and it's inertia link -->
   <link name="base_link" />
+  <link name="imu_link">
+    <inertial>
+      <mass value="0.001"/>
+      <origin rpy="0 0 0" xyz="0 0 0"/>
+      <inertia ixx="0.0001" ixy="0" ixz="0" iyy="0.000001" iyz="0" izz="0.0001"/>
+    </inertial>
+    <visual>
+      <origin rpy="0 0 0" xyz="0 0 0"/>
+      <geometry>
+        <box size="0.001 0.001 0.001"/>
+      </geometry>
+    </visual>
+    <collision>
+      <origin rpy="0 0 0" xyz="0 0 0"/>
+      <geometry>
+        <box size=".001 .001 .001"/>
+      </geometry>
+    </collision>
+  </link>
   <link name="chassis">
     <visual>
       <xacro:chassis_geometry/>
-      <!--material name="blue" /-->
     </visual>
   </link>
@@ -108,5 +126,5 @@
     </visual>
   </link>
-  <joint name="right_steering_hinge_joint" type="continuous">
+  <joint name="right_steering_hinge_joint" type="revolute">
     <origin xyz="0.25 -0.12 0" rpy="0 1.5708 0" />
     <parent link="chassis" />
@@ -160,5 +178,11 @@
   </joint>
   <xacro:wheel_transmission name="right_front_wheel" />
-  <xacro:arg name="name" default="camera" />
+  <joint name="imu_joint" type="fixed">
+    <axis xyz="1 0 0"/> <!-- 0 1 0 -->
+    <origin xyz="0 0 0.19"/>
+    <parent link="base_link"/>
+    <child link="imu_link"/>
+  </joint>
+  <!--xacro:arg name="name" default="camera" />
   <xacro:arg name="topics_ns" default="camera" />
   <xacro:arg name="use_nominal_extrinsics" default="true" />
@@ -169,15 +193,15 @@
   <xacro:sensor_d435 name="$(arg name)" topics_ns="$(arg topics_ns)" parent="realsense" use_nominal_extrinsics="$(arg use_nominal_extrinsics)" publish_pointcloud="$(arg publish_pointcloud)" add_plug="$(arg add_plug)">
     <origin xyz="0 0 0" rpy="0 0 0"/>
-  </xacro:sensor_d435>
+  </xacro:sensor_d435-->
  <!--xacro:include filename="$(find realsense2_description)/urdf/_d435.urdf.xacro">
    <sensor_d435 parent="realsense_link">
    </sensor_d435>
  </xacro:include-->
- <joint name="realsense_joint" type="fixed">
+ <!--joint name="realsense_joint" type="fixed">
    <origin xyz="0.2 0.0 0.15" rpy="0 0 0"/>
    <parent link="chassis" />
    <child link="realsense" />
    <axis xyz="0 0 1" />
- </joint>
+ </joint-->
   <!-- Add Hokuyo laser scanner -->
   <link name="laser">
@@ -205,29 +229,4 @@
     <axis xyz="0 0 1" />
   </joint>
-<joint name="imu_joint" type="fixed">
-  <axis xyz="1 0 0"/> <!-- 0 1 0 -->
-  <origin xyz="0 0 0.19"/>
-  <parent link="base_link"/>
-  <child link="imu_link"/>
-</joint>
-<link name="imu_link">
-  <inertial>
-    <mass value="0.001"/>
-    <origin rpy="0 0 0" xyz="0 0 0"/>
-    <inertia ixx="0.0001" ixy="0" ixz="0" iyy="0.000001" iyz="0" izz="0.0001"/>
-  </inertial>
-  <visual>
-    <origin rpy="0 0 0" xyz="0 0 0"/>
-    <geometry>
-      <box size="0.001 0.001 0.001"/>
-    </geometry>
-  </visual>
-  <collision>
-    <origin rpy="0 0 0" xyz="0 0 0"/>
-    <geometry>
-      <box size=".001 .001 .001"/>
-    </geometry>
-  </collision>
-</link>
 <joint name="gps_joint" type="fixed">
   <axis xyz="1 0 0"/> <!-- 0 1 0 -->
