Commit message: initial commit of car model with VESC spd controller

File: rover_description/urdf/macros.xacro (robot description, xacro)
@@ -4,5 +4,5 @@
 <xacro:macro name="chassis_inertial_params">
   <origin xyz="0.1477 0 0" rpy="0 0 0" />
-  <mass value="4.0" />
+  <mass value="5.0" />
   <inertia ixx="0.010609" ixy="0"          ixz="0"
                           iyy="0.050409"   iyz="0"
@@ -18,15 +18,19 @@
 <xacro:macro name="left_wheels_inertial_params">
   <origin xyz="0 0 -0.0225" rpy="0 0 0" />
-  <mass value="0.34055" />
+  <mass value="0.6811" />
+  <!--mass value="0.34055" /-->
   <inertia ixx="0.00026046" ixy="0"          ixz="0"
                             iyy="0.00026046" iyz="0"
-                                             izz="0.00041226" />
+                                             izz="0.0041226" />
+                                             <!--izz="0.00041226" /-->
 </xacro:macro>
 <xacro:macro name="right_wheels_inertial_params">
   <origin xyz="0 0 0.0225" rpy="0 0 0" />
-  <mass value="0.34055" />
+  <mass value="0.6811" />
+  <!--mass value="0.34055" /-->
   <inertia ixx="0.00026046" ixy="0"          ixz="0"
                             iyy="0.00026046" iyz="0"
-                                             izz="0.00041226" />
+                                             izz="0.0041226" />
+                                             <!--izz="0.00041226" /-->
 </xacro:macro>
 <xacro:macro name="steering_hinge_inertial_params">

File: rover_description/urdf/rover.xacro (robot description, xacro)
@@ -54,5 +54,5 @@
     <child link="left_rear_wheel" />
     <axis xyz="0 0 -1" />
-    <!--dynamics damping="0.05" friction="0.0"/-->
+    <dynamics damping="0.05" friction="0.0"/>
     <limit effort="10" velocity="100" />
   </joint>
@@ -76,5 +76,5 @@
     <child link="right_rear_wheel" />
     <axis xyz="0 0 -1" />
-    <!--dynamics damping="0.05" friction="0.0"/-->
+    <dynamics damping="0.05" friction="0.0"/>
     <limit effort="10" velocity="100" />
   </joint>
@@ -160,5 +160,5 @@
   </joint>
   <xacro:wheel_transmission name="right_front_wheel" />
-  <xacro:arg name="name" default="camera" />
+  <!--xacro:arg name="name" default="camera" />
   <xacro:arg name="topics_ns" default="camera" />
   <xacro:arg name="use_nominal_extrinsics" default="true" />
@@ -170,14 +170,14 @@
     <origin xyz="0 0 0" rpy="0 0 0"/>
   </xacro:sensor_d435>
- <!--xacro:include filename="$(find realsense2_description)/urdf/_d435.urdf.xacro">
+ <xacro:include filename="$(find realsense2_description)/urdf/_d435.urdf.xacro">
    <sensor_d435 parent="realsense_link">
    </sensor_d435>
  </xacro:include-->
- <joint name="realsense_joint" type="fixed">
+ <!--joint name="realsense_joint" type="fixed">
    <origin xyz="0.2 0.0 0.15" rpy="0 0 0"/>
    <parent link="chassis" />
    <child link="realsense" />
    <axis xyz="0 0 1" />
- </joint>
+ </joint-->
   <!-- Add Hokuyo laser scanner -->
   <link name="laser">

Commit message: Fixed Odom Pub Fixed Frame must be map

File: rover_description/urdf/macros.xacro (robot description, xacro)
@@ -4,8 +4,8 @@
 <xacro:macro name="chassis_inertial_params">
   <origin xyz="0.1477 0 0" rpy="0 0 0" />
-  <mass value="5.0" />
+  <mass value="10.0" />
   <inertia ixx="0.010609" ixy="0"          ixz="0"
-                          iyy="0.050409"   iyz="0"
-                                           izz="0.05865" />
+                          iyy="0.1"   iyz="0"
+                                           izz="0.1" />
 </xacro:macro>
 <xacro:macro name="body_inertial_params">
@@ -20,6 +20,6 @@
   <mass value="0.6811" />
   <!--mass value="0.34055" /-->
-  <inertia ixx="0.00026046" ixy="0"          ixz="0"
-                            iyy="0.00026046" iyz="0"
+  <inertia ixx="0.0026046" ixy="0"          ixz="0"
+                            iyy="0.0026046" iyz="0"
                                              izz="0.0041226" />
                                              <!--izz="0.00041226" /-->
@@ -29,6 +29,6 @@
   <mass value="0.6811" />
   <!--mass value="0.34055" /-->
-  <inertia ixx="0.00026046" ixy="0"          ixz="0"
-                            iyy="0.00026046" iyz="0"
+  <inertia ixx="0.0026046" ixy="0"          ixz="0"
+                            iyy="0.0026046" iyz="0"
                                              izz="0.0041226" />
                                              <!--izz="0.00041226" /-->
